File: frambuesa-rev-a/frambuesa-rev-a.kicad_sch (KiCad schematic)
At the start: 34 parts, among them J1 USB_B_Micro, J2 Conn_01x02, J3 Conn_02x18_Odd_Even, J4 Conn_02x18_Odd_Even, U1 RP2040, U2 NCP1117-3.3_SOT223, U3 W25Q128JVS, Y1 Crystal_GND24

Commit message: avanzados lcsc
Parts:
- removed C14: 100n, Capacitor_SMD:C_0805_2012Metric, symbol Device:C
- removed J1: USB_B_Micro, symbol Connector:USB_B_Micro
- removed J2: Conn_01x02, symbol Connector_Generic:Conn_01x02
- removed U2: NCP1117-3.3_SOT223, Package_TO_SOT_SMD:SOT-223-3_TabPin2, symbol Regulator_Linear:NCP1117-3.3_SOT223
- added C18: 100u, symbol Device:C
- added C19, C20: 10u, symbol Device:C
- added J5: USB_C_Receptacle_USB2.0_16P, symbol Connector:USB_C_Receptacle_USB2.0_16P
- added R6, R7: 5k1, symbol Device:R
- added SW1: PTS 636, symbol Switch:SW_SPST
- added U2: AMS1117-5.0, Package_TO_SOT_SMD:SOT-223-3_TabPin2, symbol Regulator_Linear:AMS1117-5.0
- C12: value 10u -> 100u; footprint Capacitor_SMD:CP_Elec_4x5.4 -> (none); LCSC (none) -> C15008
- C13: footprint Capacitor_SMD:CP_Elec_4x5.4 -> (none); LCSC (none) -> C15525
- R3: LCSC (none) -> C11702
- R4: value DNF -> 10k; LCSC (none) -> C25744
- U3: LCSC (none) -> C97521
Connections:
- net +3V3: now also C20.1; no longer C13.1
- net GND: now also C18.2, C19.2, C20.2, J5.A1 (GND), J5.A12 (GND), J5.B1 (GND), J5.B12 (GND), J5.SH (SHIELD), R6.2, R7.2, SW1.1 (A), U2.1 (GND)
- net NOT_QSPI_SS: no longer R3.2, R4.2, U3.1 (~{CS})
- net VBUS: now also J5.A4 (VBUS), J5.A9 (VBUS), J5.B4 (VBUS), J5.B9 (VBUS); no longer C12.1
- net at R3.1: now also SW1.2 (B)
- new net: J5.A5 (CC1), R6.1
- new net: J5.B5 (CC2), R7.1
- new net +3.3V: C18.1, C19.1, U2.2 (VO)
- new net QSPI_SS: R3.2, R4.2, U3.1 (~{CS})
- new net USB_D+: J5.A6 (D+), J5.B6 (D+)
- new net USB_D-: J5.A7 (D-), J5.B7 (D-)
- new net VHI: C12.1, C13.1, U2.3 (VI)
- no-connect marks 1 -> 2
Other:
- note added: "TODO ordenar de otra manera"
- note added: "boot"
- note added: "cristal TODO"
- note added: "flash FP pending"
- note added: "poder FP pending"
- note added: "usb FP pending"
- note removed: "cristal"
- note removed: "flash"
- note removed: "poder"
- moved on the sheet: R3, R4
