File: frambuesa-rev-a/frambuesa-rev-a.kicad_sch (KiCad schematic)
At the start: 34 parts, among them J1 USB_B_Micro, J2 Conn_01x02, J3 Conn_02x18_Odd_Even, J4 Conn_02x18_Odd_Even, U1 RP2040, U2 NCP1117-3.3_SOT223, U3 W25Q128JVS, Y1 Crystal_GND24

Commit message: agregar usb-c y cajitas
Parts:
- removed H1, H2, H3, H4: MountingHole, MountingHole:MountingHole_3.2mm_M3, symbol Mechanical:MountingHole
- removed J1: USB_B_Micro, symbol Connector:USB_B_Micro
- removed J3, J4: Conn_02x18_Odd_Even, Connector_PinSocket_2.54mm:PinSocket_1x20_P2.54mm_Vertical, symbol Connector_Generic:Conn_02x18_Odd_Even
- added C18: 100u, Capacitor_SMD:CP_Elec_4x5.4, symbol Device:C
- added D1, D2: 1N5819WS, Diode_SMD:D_SOD-323, symbol Diode:1N5819WS
- added D3, D4: LED, symbol Device:LED
- added J3, J4: Conn_01x20_Pin, symbol Connector:Conn_01x20_Pin
- added J5: USB_C_Receptacle_USB2.0_16P, symbol Connector:USB_C_Receptacle_USB2.0_16P
- added R6, R7: 5.1k, symbol Device:R
- added R8, R9: 10k, symbol Device:R
- C15: value 10u -> 100u
Connections:
- net +3V3: now also C18.1, J4.16 (Pin_16), R8.1; no longer C15.1
- net GND: now also C18.2, D3.1 (K), D4.1 (K), J3.13 (Pin_13), J3.18 (Pin_18), J3.3 (Pin_3), J3.8 (Pin_8), J4.13 (Pin_13), J4.18 (Pin_18), J4.3 (Pin_3), J4.8 (Pin_8), J5.A1 (GND), J5.A12 (GND), J5.B1 (GND), J5.B12 (GND), J5.SH (SHIELD), R6.1, R7.1
- net GPIO00: now also J3.1 (Pin_1)
- net GPIO01: now also J3.2 (Pin_2)
- net GPIO02: now also J3.4 (Pin_4)
- net GPIO03: now also J3.5 (Pin_5)
- net GPIO04: now also J3.6 (Pin_6)
- net GPIO05: now also J3.7 (Pin_7)
- net GPIO06: now also J3.9 (Pin_9)
- net GPIO07: now also J3.10 (Pin_10)
- net GPIO08: now also J3.11 (Pin_11)
- net GPIO09: now also J3.12 (Pin_12)
- net GPIO10: now also J3.14 (Pin_14)
- net GPIO11: now also J3.15 (Pin_15)
- net GPIO12: now also J3.16 (Pin_16)
- net GPIO13: now also J3.17 (Pin_17)
- net GPIO14: now also J3.19 (Pin_19), R9.1
- net GPIO15: now also J3.20 (Pin_20)
- net GPIO16: now also J4.1 (Pin_1)
- net GPIO17: now also J4.2 (Pin_2)
- net GPIO18: now also J4.4 (Pin_4)
- net GPIO19: now also J4.5 (Pin_5)
- net GPIO20: now also J4.6 (Pin_6)
- net GPIO21: now also J4.7 (Pin_7)
- net GPIO22: now also J4.9 (Pin_9)
- net GPIO26_ADC0: now also J4.11 (Pin_11)
- net GPIO27_ADC1: now also J4.12 (Pin_12)
- net GPIO28_ADC2: now also J4.14 (Pin_14)
- net RUN: now also J4.10 (Pin_10)
- net USB_D_MINUS: now also J5.A7 (D-), J5.B7 (D-)
- net USB_D_PLUS: now also J5.A6 (D+), J5.B6 (D+)
- net VBUS: now also D1.2 (A), J5.A4 (VBUS), J5.A9 (VBUS), J5.B4 (VBUS), J5.B9 (VBUS); no longer C12.1, U2.3 (VI)
- net XOUT: now also R5.1; no longer R5.2
- net at C17.2, Y1.3: now also R5.2; no longer R5.1
- new net: D3.2 (A), R8.2
- new net: J5.A5 (CC1), R6.2
- new net: J5.B5 (CC2), R7.2
- new net: D4.2 (A), R9.2
- new net VHI: C12.1, C15.1, D1.1 (K), D2.1 (K), U2.3 (VI)
- new net VIN: D2.2 (A)
- no-connect marks 1 -> 2
Other:
- note added: "leds"
- note added: "usb"

Commit message: commit
Parts:
- removed C14: 100n, Capacitor_SMD:C_0805_2012Metric, symbol Device:C
- removed D1, D2: 1N5819WS, Diode_SMD:D_SOD-323, symbol Diode:1N5819WS
- removed D3, D4: LED, symbol Device:LED
- removed J2: Conn_01x02, symbol Connector_Generic:Conn_01x02
- removed J3, J4: Conn_01x20_Pin, symbol Connector:Conn_01x20_Pin
- removed R8, R9: 10k, symbol Device:R
- removed U2: NCP1117-3.3_SOT223, Package_TO_SOT_SMD:SOT-223-3_TabPin2, symbol Regulator_Linear:NCP1117-3.3_SOT223
- added C19, C20: 10u, symbol Device:C
- added H1, H2, H3, H4: MountingHole, MountingHole:MountingHole_3.2mm_M3, symbol Mechanical:MountingHole
- added J3, J4: Conn_02x18_Odd_Even, Connector_PinSocket_2.54mm:PinSocket_1x20_P2.54mm_Vertical, symbol Connector_Generic:Conn_02x18_Odd_Even
- added SW1: PTS 636, symbol Switch:SW_SPST
- added U2: AMS1117-5.0, Package_TO_SOT_SMD:SOT-223-3_TabPin2, symbol Regulator_Linear:AMS1117-5.0
- C12: value 10u -> 100u; footprint Capacitor_SMD:CP_Elec_4x5.4 -> (none); LCSC (none) -> C15008
- C13: footprint Capacitor_SMD:CP_Elec_4x5.4 -> (none); LCSC (none) -> C15525
- C15: value 100u -> 10u
- C18: footprint Capacitor_SMD:CP_Elec_4x5.4 -> (none); LCSC (none) -> C15008
- J5: LCSC (none) -> C165948
- R3: LCSC (none) -> C11702
- R4: value DNF -> 10k; LCSC (none) -> C25744
- R6, R7: value 5.1k -> 5k1; LCSC (none) -> C25905
- U3: LCSC (none) -> C97521
Connections:
- net +3V3: now also C15.1, C20.1, J3.2 (Pin_2); no longer C13.1, C18.1
- net GND: now also R6.2, R7.2, C19.2, C20.2, J3.1 (Pin_1), J3.11 (Pin_11), J3.13 (Pin_13), J3.15 (Pin_15), J3.17 (Pin_17), J3.19 (Pin_19), J3.21 (Pin_21), J3.23 (Pin_23), J3.25 (Pin_25), J3.27 (Pin_27), J3.29 (Pin_29), J3.3 (Pin_3), J3.31 (Pin_31), J3.33 (Pin_33), J3.35 (Pin_35), J3.36 (Pin_36), J3.5 (Pin_5), J3.7 (Pin_7), J3.9 (Pin_9), J4.10 (Pin_10), J4.12 (Pin_12), J4.14 (Pin_14), J4.16 (Pin_16), J4.18 (Pin_18), J4.2 (Pin_2), J4.20 (Pin_20), J4.22 (Pin_22), J4.24 (Pin_24), J4.26 (Pin_26), J4.28 (Pin_28), J4.30 (Pin_30), J4.32 (Pin_32), J4.34 (Pin_34), J4.35 (Pin_35), J4.36 (Pin_36), J4.4 (Pin_4), J4.6 (Pin_6), J4.8 (Pin_8), SW1.1 (A), U2.1 (GND); no longer R6.1, R7.1
- net GPIO00: now also J3.4 (Pin_4)
- net GPIO01: now also J3.6 (Pin_6)
- net GPIO02: now also J3.8 (Pin_8)
- net GPIO03: now also J3.10 (Pin_10)
- net GPIO04: now also J3.12 (Pin_12)
- net GPIO05: now also J3.14 (Pin_14)
- net GPIO06: now also J3.16 (Pin_16)
- net GPIO07: now also J3.18 (Pin_18)
- net GPIO08: now also J3.20 (Pin_20)
- net GPIO09: now also J3.22 (Pin_22)
- net GPIO10: now also J3.24 (Pin_24)
- net GPIO11: now also J3.26 (Pin_26)
- net GPIO12: now also J3.28 (Pin_28)
- net GPIO13: now also J3.30 (Pin_30)
- net GPIO14: now also J3.32 (Pin_32)
- net GPIO15: now also J3.34 (Pin_34)
- net GPIO16: now also J4.27 (Pin_27)
- net GPIO17: now also J4.25 (Pin_25)
- net GPIO18: now also J4.23 (Pin_23)
- net GPIO19: now also J4.21 (Pin_21)
- net GPIO20: now also J4.19 (Pin_19)
- net GPIO21: now also J4.17 (Pin_17)
- net GPIO22: now also J4.15 (Pin_15)
- net GPIO23: now also J4.13 (Pin_13)
- net GPIO24: now also J4.11 (Pin_11)
- net GPIO25: now also J4.9 (Pin_9)
- net GPIO26_ADC0: now also J4.7 (Pin_7)
- net GPIO27_ADC1: now also J4.5 (Pin_5)
- net GPIO28_ADC2: now also J4.3 (Pin_3)
- net GPIO29_ADC3: now also J4.1 (Pin_1)
- net NOT_QSPI_SS: no longer R3.2, R4.2, U3.1 (~{CS})
- net RUN: now also J4.29 (Pin_29)
- net SWCLK: now also J4.33 (Pin_33)
- net SWD: now also J4.31 (Pin_31)
- net USB_D_MINUS: no longer J5.A7 (D-), J5.B7 (D-)
- net USB_D_PLUS: no longer J5.A6 (D+), J5.B6 (D+)
- net VHI: now also C13.1, U2.3 (VI); no longer C15.1
- net XOUT: now also R5.2; no longer R5.1
- net at R3.1: now also SW1.2 (B)
- net at C17.2, Y1.3: now also R5.1; no longer R5.2
- net at J5.A5 (CC1): now also R6.1; no longer R6.2
- net at J5.B5 (CC2): now also R7.1; no longer R7.2
- new net +3.3V: C18.1, C19.1, U2.2 (VO)
- new net QSPI_SS: R3.2, R4.2, U3.1 (~{CS})
- new net USB_D+: J5.A6 (D+), J5.B6 (D+)
- new net USB_D-: J5.A7 (D-), J5.B7 (D-)
Other:
- note added: "TODO ordenar de otra manera"
- note added: "boot"
- note added: "cristal TODO"
- note added: "flash FP pending"
- note added: "poder FP pending"
- note added: "usb FP pending"
- note removed: "cristal"
- note removed: "flash"
- note removed: "leds"
- note removed: "poder"
- note removed: "usb"
- moved on the sheet: R3, R4

Commit message: agregar borrador de biblioteca local para proyecto
Other:
- title: (none) -> frambuesa
Changed lines of the file:
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@@
 	(paper "A3" portrait)
 	(title_block
+		(title "frambuesa")
+		(date "2026-09-17")
+		(rev "rev-a")
 		(company "piruetas SpA")
 	)
